File: hw/felderblock/Felderblock_Hebelplatine.brd (EAGLE design)
At the start: 50 x 78 mm, 35 parts, among them IC3 MCP23017SP

Commit message: added names
Routing:
- net FST6_LED: track 44.0 -> 45.9 mm
- net FST4_LED: track 58.3 -> 59.4 mm
- net FST8_LED: track 71.0 -> 72.0 mm
Other:
- board text added: "Felderblock Hebelplatine v1 DKap/JBec 2021"
