File: hw/felderblock/Felderblock_Grundplatine.sch (EAGLE design)
At the start: 47 parts, among them IC1 LM311N, IC2 LM2936Z-5.0, J1 RJ11, J2 RJ11, M1 ARDUINO-NANO-3.0, T1 BC337, X1 TASTENSPERRE1, X2 TASTENSPERRE2, X3 SCHLUESSELSPERRE, X4 I2C

Commit message: MI+AsT integrated
LED nach I2C, MI links und rechts, AsT und AsM integriert. Board rerouted
Parts:
- removed IC1: LM311N, linear:LM311N
- removed R1: 22k, resistor:R-EU_0207/10
- removed R2: 10k, resistor:R-EU_0207/10
- removed R3: 150k, resistor:R-EU_0207/10
- removed R4: 47k, resistor:R-EU_0207/10
- removed R5: 220k, resistor:R-EU_0207/10
- removed R6: 2.2k, resistor:R-EU_0207/10
- removed T1: BC337, transistor:BC337
- added C6: 47pF, resistor:C-EU025-024X044
- added C7: 1nF, resistor:C-EU025-025X050
- added IC4: MCP2300X/P, adafruit:MCP2300X/P
- added R15: 1k, resistor:R-EU_0207/7
- added R16, R17: 12R, resistor:R-EU_0207/7
- added R18: 130K, resistor:R-EU_0207/7
- added R19: 47k, resistor:R-EU_0207/7
- added R20: 3K3, resistor:R-EU_0207/7
- added S5, S6: EC11B42AE, alps:EC11B42AE
- added T2: BC337, transistor:BC337
- added X5: ANSCHALTER, con-molex:22-23-2041
Connections:
- removed net N$1: IC1.-IN, R1.2, R2.1
- removed net N$18: IC3.I7
- removed net N$2: R6.2, T1.B
- removed net N$26: IC3.O7
- removed net N$3: IC1.+IN, R3.2, R4.1, R5.2
- new net AS_LED: IC3.I7, IC4.GP6
- new net AS_LEDD: IC3.O7, X5-3.S
- new net AS_SW: M1.A3, X5-4.S
- new net BASE: C7.2, R20.2, T2.B
- new net LN_INTERN: R17.2, R18.2, T2.C
- new net MI_FWD: M1.D6, S5W.B, S6W.B
- new net MI_SW: M1.D5, S5G$3.D, S6G$3.D
- new net N$11: C6.1, R16.2, R17.1
- net +5V: now also IC4.A0, IC4.VCC, R15.2, X5-2.S; no longer IC1.V+, R2.2
- net FELD1_LED: now also IC4.GP0; no longer M1.D3
- net FELD2_LED: now also IC4.GP1; no longer M1.D4
- net FELD3_LED: now also IC4.GP2; no longer M1.D5
- net FELD4_LED: now also IC4.GP3; no longer M1.D6
- net GND: now also C6.2, IC4./RST, IC4.A1, IC4.A2, IC4.GND, IC4.INT, M1.GND.2, R15.1, R19.1, S5G$3.E, S5W.C, S5W.GND, S6G$3.E, S6W.C, S6W.GND, T2.E, X5-1.S; no longer IC1.GND, IC1.V-, R1.1, R3.1, T1.E
- net LN_RX: now also R18.1, R19.2; no longer IC1.OUT, R5.1
- net LN_TX: now also C7.1, R20.1; no longer R6.1
- net LOCONET: now also R16.1; no longer R4.2, T1.C
- net SCL: now also IC4.SCL
- net SDA: now also IC4.SDA
- net TSP1_LED: now also IC4.GP4; no longer M1.A0
- net TSP2_LED: now also IC4.GP5; no longer M1.A2
- net TSP2_SW: now also M1.A2; no longer M1.A3

Commit message: Changed pin order on MCP
MCP moved to other side, changed pin order
Parts:
- IC3: value (none) -> ULN2803
Connections:
- net AS_LED: now also IC4.GP1; no longer IC4.GP6
- net FELD1_LED: now also IC4.GP7; no longer IC4.GP0
- net FELD2_LED: now also IC4.GP6; no longer IC4.GP1
- net FELD3_LED: now also IC4.GP5; no longer IC4.GP2
- net FELD4_LED: now also IC4.GP4; no longer IC4.GP3
- net TSP1_LED: now also IC4.GP3; no longer IC4.GP4
- net TSP2_LED: now also IC4.GP2; no longer IC4.GP5
Changed lines of the file:
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@@
 <?xml version="1.0" encoding="utf-8"?>
 <!DOCTYPE eagle SYSTEM "eagle.dtd">
-<eagle version="7.6.0">
+<eagle version="7.3.0">
 <drawing>
 <settings>
@@
 <part name="X2" library="con-molex" deviceset="22-23-2041" device="" value="TASTENSPERRE2"/>
 <part name="X3" library="con-molex" deviceset="22-23-2021" device="" value="SCHLUESSELSPERRE"/>
-<part name="IC3" library="uln-udn" deviceset="ULN2803A" device="DIL18"/>
+<part name="IC3" library="uln-udn" deviceset="ULN2803A" device="DIL18" value="ULN2803"/>
 <part name="GND13" library="supply1" deviceset="GND" device=""/>
 <part name="P+5" library="supply1" deviceset="+5V" device=""/>
@@
 </segment>
 <segment>
-<pinref part="IC4" gate="G$1" pin="GP0"/>
-<wire x1="167.64" y1="76.2" x2="190.5" y2="76.2" width="0.1524" layer="91"/>
-<label x="175.26" y="76.2" size="1.778" layer="95"/>
+<pinref part="IC4" gate="G$1" pin="GP7"/>
+<wire x1="190.5" y1="58.42" x2="167.64" y2="58.42" width="0.1524" layer="91"/>
+<label x="172.72" y="58.42" size="1.778" layer="95"/>
 </segment>
 </net>
@@
 </segment>
 <segment>
-<pinref part="IC4" gate="G$1" pin="GP1"/>
-<wire x1="167.64" y1="73.66" x2="190.5" y2="73.66" width="0.1524" layer="91"/>
-<label x="175.26" y="73.66" size="1.778" layer="95"/>
+<pinref part="IC4" gate="G$1" pin="GP6"/>
+<wire x1="190.5" y1="60.96" x2="167.64" y2="60.96" width="0.1524" layer="91"/>
+<label x="172.72" y="60.96" size="1.778" layer="95"/>
 </segment>
 </net>
@@
 </segment>
 <segment>
-<pinref part="IC4" gate="G$1" pin="GP3"/>
-<wire x1="167.64" y1="68.58" x2="190.5" y2="68.58" width="0.1524" layer="91"/>
-<label x="175.26" y="68.58" size="1.778" layer="95"/>
+<pinref part="IC4" gate="G$1" pin="GP4"/>
+<wire x1="190.5" y1="66.04" x2="167.64" y2="66.04" width="0.1524" layer="91"/>
+<label x="172.72" y="66.04" size="1.778" layer="95"/>
 </segment>
 </net>
@@
 </segment>
 <segment>
-<pinref part="IC4" gate="G$1" pin="GP2"/>
-<wire x1="167.64" y1="71.12" x2="190.5" y2="71.12" width="0.1524" layer="91"/>
-<label x="175.26" y="71.12" size="1.778" layer="95"/>
+<pinref part="IC4" gate="G$1" pin="GP5"/>
+<wire x1="190.5" y1="63.5" x2="167.64" y2="63.5" width="0.1524" layer="91"/>
+<label x="172.72" y="63.5" size="1.778" layer="95"/>
 </segment>
 </net>
@@
 </segment>
 <segment>
-<pinref part="IC4" gate="G$1" pin="GP5"/>
-<wire x1="167.64" y1="63.5" x2="190.5" y2="63.5" width="0.1524" layer="91"/>
-<label x="175.26" y="63.5" size="1.778" layer="95"/>
+<pinref part="IC4" gate="G$1" pin="GP2"/>
+<wire x1="190.5" y1="71.12" x2="167.64" y2="71.12" width="0.1524" layer="91"/>
+<label x="172.72" y="71.12" size="1.778" layer="95"/>
 </segment>
 </net>
@@
 </segment>
 <segment>
-<wire x1="167.64" y1="66.04" x2="190.5" y2="66.04" width="0.1524" layer="91"/>
-<label x="175.26" y="66.04" size="1.778" layer="95"/>
-<pinref part="IC4" gate="G$1" pin="GP4"/>
+<pinref part="IC4" gate="G$1" pin="GP3"/>
+<wire x1="190.5" y1="68.58" x2="167.64" y2="68.58" width="0.1524" layer="91"/>
+<label x="172.72" y="68.58" size="1.778" layer="95"/>
 </segment>
 </net>
@@
 <net name="AS_LED" class="0">
 <segment>
-<pinref part="IC4" gate="G$1" pin="GP6"/>
-<wire x1="167.64" y1="60.96" x2="190.5" y2="60.96" width="0.1524" layer="91"/>
-<label x="175.26" y="60.96" size="1.778" layer="95"/>
-</segment>
-<segment>
 <pinref part="IC3" gate="G$1" pin="I7"/>
 <wire x1="27.94" y1="63.5" x2="43.18" y2="63.5" width="0.1524" layer="91"/>
 <label x="27.94" y="63.5" size="1.778" layer="95"/>
 </segment>
-</net>
+<segment>
+<pinref part="IC4" gate="G$1" pin="GP1"/>
+<wire x1="190.5" y1="73.66" x2="167.64" y2="73.66" width="0.1524" layer="91"/>
+<label x="172.72" y="73.66" size="1.778" layer="95"/>
+</segment>
+</net>

Commit message: housekeeping
some reroutes, text optimized
Parts:
- IC2: value LM2936Z-5.0 -> LM2936
Connections:
- net MI_FWD: now also S5W.A, S6W.A
Other:
- moved on the sheet: S5W, S6W
Changed lines of the file:
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@@
 <?xml version="1.0" encoding="utf-8"?>
 <!DOCTYPE eagle SYSTEM "eagle.dtd">
-<eagle version="7.3.0">
+<eagle version="7.6.0">
 <drawing>
 <settings>
@@
 <part name="D2" library="diode" deviceset="1N581*" device="" technology="9-T"/>
 <part name="RS" library="jumper" deviceset="JP1E" device=""/>
-<part name="IC2" library="national-semiconductor" deviceset="LM2936?*" device="Z" technology="-5.0"/>
+<part name="IC2" library="national-semiconductor" deviceset="LM2936?*" device="Z" technology="-5.0" value="LM2936"/>
 <part name="C1" library="resistor" deviceset="C-EU" device="025-025X050" value="100nF"/>
 <part name="C2" library="resistor" deviceset="C-EU" device="025-025X050" value="100nF"/>
@@
 <instance part="X4" gate="-3" x="167.64" y="99.06"/>
 <instance part="X4" gate="-4" x="167.64" y="96.52"/>
-<instance part="S5" gate="G$3" x="-55.88" y="55.88" rot="R90"/>
-<instance part="S5" gate="W" x="-55.88" y="73.66" rot="R90"/>
-<instance part="S6" gate="G$3" x="-55.88" y="81.28" rot="R90"/>
-<instance part="S6" gate="W" x="-55.88" y="48.26" rot="R90"/>
+<instance part="S5" gate="G$3" x="-73.66" y="63.5" rot="R90"/>
+<instance part="S5" gate="W" x="-73.66" y="99.06" rot="R90"/>
+<instance part="S6" gate="G$3" x="-73.66" y="106.68" rot="R90"/>
+<instance part="S6" gate="W" x="-73.66" y="55.88" rot="R90"/>
 <instance part="IC4" gate="G$1" x="152.4" y="66.04"/>
 <instance part="R15" gate="G$1" x="124.46" y="50.8" rot="R90"/>
@@
 </segment>
 <segment>
-<wire x1="-63.5" y1="73.66" x2="-68.58" y2="73.66" width="0.1524" layer="91"/>
+<wire x1="-81.28" y1="99.06" x2="-86.36" y2="99.06" width="0.1524" layer="91"/>
 <pinref part="S5" gate="W" pin="C"/>
-<label x="-73.66" y="73.66" size="1.778" layer="95"/>
+<label x="-91.44" y="99.06" size="1.778" layer="95"/>
 <pinref part="S6" gate="G$3" pin="E"/>
-<wire x1="-68.58" y1="73.66" x2="-76.2" y2="73.66" width="0.1524" layer="91"/>
-<wire x1="-60.96" y1="81.28" x2="-68.58" y2="81.28" width="0.1524" layer="91"/>
-<wire x1="-68.58" y1="81.28" x2="-68.58" y2="73.66" width="0.1524" layer="91"/>
-<junction x="-68.58" y="73.66"/>
-</segment>
-<segment>
-<wire x1="-63.5" y1="48.26" x2="-68.58" y2="48.26" width="0.1524" layer="91"/>
+<wire x1="-86.36" y1="99.06" x2="-93.98" y2="99.06" width="0.1524" layer="91"/>
+<wire x1="-78.74" y1="106.68" x2="-86.36" y2="106.68" width="0.1524" layer="91"/>
+<wire x1="-86.36" y1="106.68" x2="-86.36" y2="99.06" width="0.1524" layer="91"/>
+<junction x="-86.36" y="99.06"/>
+</segment>
+<segment>
+<wire x1="-81.28" y1="55.88" x2="-86.36" y2="55.88" width="0.1524" layer="91"/>
 <pinref part="S6" gate="W" pin="C"/>
-<label x="-73.66" y="48.26" size="1.778" layer="95"/>
+<label x="-91.44" y="55.88" size="1.778" layer="95"/>
 <pinref part="S5" gate="G$3" pin="E"/>
-<wire x1="-68.58" y1="48.26" x2="-76.2" y2="48.26" width="0.1524" layer="91"/>
-<wire x1="-60.96" y1="55.88" x2="-68.58" y2="55.88" width="0.1524" layer="91"/>
-<wire x1="-68.58" y1="55.88" x2="-68.58" y2="48.26" width="0.1524" layer="91"/>
-<junction x="-68.58" y="48.26"/>
+<wire x1="-86.36" y1="55.88" x2="-93.98" y2="55.88" width="0.1524" layer="91"/>
+<wire x1="-78.74" y1="63.5" x2="-86.36" y2="63.5" width="0.1524" layer="91"/>
+<wire x1="-86.36" y1="63.5" x2="-86.36" y2="55.88" width="0.1524" layer="91"/>
+<junction x="-86.36" y="55.88"/>
 </segment>
 <segment>
 <pinref part="S5" gate="W" pin="GND"/>
-<wire x1="-50.8" y1="66.04" x2="-33.02" y2="66.04" width="0.1524" layer="91"/>
-<label x="-43.18" y="66.04" size="1.778" layer="95"/>
+<wire x1="-68.58" y1="91.44" x2="-50.8" y2="91.44" width="0.1524" layer="91"/>
+<label x="-60.96" y="91.44" size="1.778" layer="95"/>
 </segment>
 <segment>
 <pinref part="S6" gate="W" pin="GND"/>
-<wire x1="-50.8" y1="40.64" x2="-33.02" y2="40.64" width="0.1524" layer="91"/>
-<label x="-40.64" y="40.64" size="1.778" layer="95"/>
+<wire x1="-68.58" y1="48.26" x2="-50.8" y2="48.26" width="0.1524" layer="91"/>
+<label x="-58.42" y="48.26" size="1.778" layer="95"/>
 </segment>
 <segment>
@@
 <net name="MI_FWD" class="0">
 <segment>
-<wire x1="-50.8" y1="76.2" x2="-33.02" y2="76.2" width="0.1524" layer="91"/>
 <pinref part="S5" gate="W" pin="B"/>
-<label x="-45.72" y="76.2" size="1.778" layer="95"/>
-</segment>
-<segment>
-<wire x1="-50.8" y1="50.8" x2="-33.02" y2="50.8" width="0.1524" layer="91"/>
+<label x="-63.5" y="101.6" size="1.778" layer="95"/>
+<pinref part="S5" gate="W" pin="A"/>
+<wire x1="-68.58" y1="101.6" x2="-63.5" y2="101.6" width="0.1524" layer="91"/>
+<wire x1="-63.5" y1="101.6" x2="-40.64" y2="101.6" width="0.1524" layer="91"/>
+<wire x1="-68.58" y1="96.52" x2="-63.5" y2="96.52" width="0.1524" layer="91"/>
+<wire x1="-63.5" y1="96.52" x2="-63.5" y2="101.6" width="0.1524" layer="91"/>
+<junction x="-63.5" y="101.6"/>
+</segment>
+<segment>
 <pinref part="S6" gate="W" pin="B"/>
-<label x="-45.72" y="50.8" size="1.778" layer="95"/>
+<label x="-63.5" y="58.42" size="1.778" layer="95"/>
+<pinref part="S6" gate="W" pin="A"/>
+<wire x1="-68.58" y1="58.42" x2="-63.5" y2="58.42" width="0.1524" layer="91"/>
+<wire x1="-63.5" y1="58.42" x2="-50.8" y2="58.42" width="0.1524" layer="91"/>
+<wire x1="-68.58" y1="53.34" x2="-63.5" y2="53.34" width="0.1524" layer="91"/>
+<wire x1="-63.5" y1="53.34" x2="-63.5" y2="58.42" width="0.1524" layer="91"/>
+<junction x="-63.5" y="58.42"/>
 </segment>
 <segment>
@@
 <segment>
 <pinref part="S6" gate="G$3" pin="D"/>
-<wire x1="-50.8" y1="81.28" x2="-30.48" y2="81.28" width="0.1524" layer="91"/>
-<label x="-45.72" y="81.28" size="1.778" layer="95"/>
+<wire x1="-68.58" y1="106.68" x2="-48.26" y2="106.68" width="0.1524" layer="91"/>
+<label x="-63.5" y="106.68" size="1.778" layer="95"/>
 </segment>
 <segment>
 <pinref part="S5" gate="G$3" pin="D"/>
-<wire x1="-50.8" y1="55.88" x2="-33.02" y2="55.88" width="0.1524" layer="91"/>
-<label x="-45.72" y="55.88" size="1.778" layer="95"/>
-</segment>
-</net>
+<wire x1="-68.58" y1="63.5" x2="-50.8" y2="63.5" width="0.1524" layer="91"/>
+<label x="-63.5" y="63.5" size="1.778" layer="95"/>
+</segment>
+</net>

Commit message: CW and CCW split
Connections:
- new net MI_REV: M1.D5, S5W.A, S6W.A
- net MI_FWD: no longer S5W.A, S6W.A
- net MI_SW: now also M1.D4; no longer M1.D5
Changed lines of the file:
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@@
 <pinref part="S5" gate="W" pin="B"/>
 <label x="-63.5" y="101.6" size="1.778" layer="95"/>
-<pinref part="S5" gate="W" pin="A"/>
-<wire x1="-68.58" y1="101.6" x2="-63.5" y2="101.6" width="0.1524" layer="91"/>
-<wire x1="-63.5" y1="101.6" x2="-40.64" y2="101.6" width="0.1524" layer="91"/>
-<wire x1="-68.58" y1="96.52" x2="-63.5" y2="96.52" width="0.1524" layer="91"/>
-<wire x1="-63.5" y1="96.52" x2="-63.5" y2="101.6" width="0.1524" layer="91"/>
-<junction x="-63.5" y="101.6"/>
+<wire x1="-68.58" y1="101.6" x2="-50.8" y2="101.6" width="0.1524" layer="91"/>
 </segment>
 <segment>
 <pinref part="S6" gate="W" pin="B"/>
 <label x="-63.5" y="58.42" size="1.778" layer="95"/>
-<pinref part="S6" gate="W" pin="A"/>
-<wire x1="-68.58" y1="58.42" x2="-63.5" y2="58.42" width="0.1524" layer="91"/>
-<wire x1="-63.5" y1="58.42" x2="-50.8" y2="58.42" width="0.1524" layer="91"/>
-<wire x1="-68.58" y1="53.34" x2="-63.5" y2="53.34" width="0.1524" layer="91"/>
-<wire x1="-63.5" y1="53.34" x2="-63.5" y2="58.42" width="0.1524" layer="91"/>
-<junction x="-63.5" y="58.42"/>
+<wire x1="-68.58" y1="58.42" x2="-50.8" y2="58.42" width="0.1524" layer="91"/>
 </segment>
 <segment>
@@
 <net name="MI_SW" class="0">
 <segment>
-<pinref part="M1" gate="G$1" pin="D5"/>
-<wire x1="195.58" y1="162.56" x2="213.36" y2="162.56" width="0.1524" layer="91"/>
-<label x="200.66" y="162.56" size="1.778" layer="95"/>
-</segment>
-<segment>
 <pinref part="S6" gate="G$3" pin="D"/>
-<wire x1="-68.58" y1="106.68" x2="-48.26" y2="106.68" width="0.1524" layer="91"/>
+<wire x1="-68.58" y1="106.68" x2="-50.8" y2="106.68" width="0.1524" layer="91"/>
 <label x="-63.5" y="106.68" size="1.778" layer="95"/>
 </segment>
@@
 <wire x1="-68.58" y1="63.5" x2="-50.8" y2="63.5" width="0.1524" layer="91"/>
 <label x="-63.5" y="63.5" size="1.778" layer="95"/>
+</segment>
+<segment>
+<pinref part="M1" gate="G$1" pin="D4"/>
+<wire x1="195.58" y1="160.02" x2="213.36" y2="160.02" width="0.1524" layer="91"/>
+<label x="200.66" y="160.02" size="1.778" layer="95"/>
 </segment>
 </net>
@@
 </segment>
 </net>
+<net name="MI_REV" class="0">
+<segment>
+<pinref part="M1" gate="G$1" pin="D5"/>
+<wire x1="195.58" y1="162.56" x2="213.36" y2="162.56" width="0.1524" layer="91"/>
+<label x="200.66" y="162.56" size="1.778" layer="95"/>
+</segment>
+<segment>
+<pinref part="S5" gate="W" pin="A"/>
+<wire x1="-68.58" y1="96.52" x2="-50.8" y2="96.52" width="0.1524" layer="91"/>
+<label x="-63.5" y="96.52" size="1.778" layer="95"/>
+</segment>
+<segment>
+<pinref part="S6" gate="W" pin="A"/>
+<wire x1="-68.58" y1="53.34" x2="-50.8" y2="53.34" width="0.1524" layer="91"/>
+<label x="-63.5" y="53.34" size="1.778" layer="95"/>
+</segment>
+</net>

Commit message: changed I2C connectors
Parts:
- removed X4: I2C, con-molex:22-23-2041
- added I2C: (no value), SparkFun-Connectors:CONN_04JST-PTH-VERT
Connections:
- net +5V: now also I2C.3; no longer X4-2.S
- net GND: now also I2C.4; no longer X4-1.S
- net SCL: now also I2C.1; no longer X4-4.S
- net SDA: now also I2C.2; no longer X4-3.S
Changed lines of the file:
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@@
 <?xml version="1.0" encoding="utf-8"?>
 <!DOCTYPE eagle SYSTEM "eagle.dtd">
-<eagle version="7.6.0">
+<eagle version="7.7.0">
 <drawing>
 <settings>
@@
 <part name="GND13" library="supply1" deviceset="GND" device=""/>
 <part name="P+5" library="supply1" deviceset="+5V" device=""/>
-<part name="X4" library="con-molex" deviceset="22-23-2041" device="" value="I2C"/>
 <part name="S5" library="alps" deviceset="EC11B42AE" device=""/>
 <part name="S6" library="alps" deviceset="EC11B42AE" device=""/>
@@
 <part name="GND15" library="supply1" deviceset="GND" device=""/>
 <part name="GND16" library="supply1" deviceset="GND" device=""/>
+<part name="I2C" library="SparkFun-Connectors" deviceset="CONN_04" device="JST-PTH-VERT"/>
 </parts>
 <sheets>
@@
 <instance part="GND13" gate="1" x="27.94" y="48.26"/>
 <instance part="P+5" gate="1" x="88.9" y="55.88"/>
-<instance part="X4" gate="-1" x="167.64" y="104.14"/>
-<instance part="X4" gate="-2" x="167.64" y="101.6"/>
-<instance part="X4" gate="-3" x="167.64" y="99.06"/>
-<instance part="X4" gate="-4" x="167.64" y="96.52"/>
 <instance part="S5" gate="G$3" x="-73.66" y="63.5" rot="R90"/>
 <instance part="S5" gate="W" x="-73.66" y="99.06" rot="R90"/>
@@
 <instance part="GND15" gate="1" x="-121.92" y="10.16"/>
 <instance part="GND16" gate="1" x="-68.58" y="10.16"/>
+<instance part="I2C" gate="J1" x="170.18" y="99.06" rot="MR0"/>
 </instances>
 <busses>
@@
 <wire x1="149.86" y1="104.14" x2="165.1" y2="104.14" width="0.1524" layer="91"/>
 <label x="152.4" y="104.14" size="1.778" layer="95"/>
-<pinref part="X4" gate="-1" pin="S"/>
+<pinref part="I2C" gate="J1" pin="4"/>
 </segment>
 <segment>
@@
 <wire x1="149.86" y1="101.6" x2="165.1" y2="101.6" width="0.1524" layer="91"/>
 <label x="152.4" y="101.6" size="1.778" layer="95"/>
-<pinref part="X4" gate="-2" pin="S"/>
+<pinref part="I2C" gate="J1" pin="3"/>
 </segment>
 <segment>
@@
 <wire x1="149.86" y1="99.06" x2="165.1" y2="99.06" width="0.1524" layer="91"/>
 <label x="152.4" y="99.06" size="1.778" layer="95"/>
-<pinref part="X4" gate="-3" pin="S"/>
+<pinref part="I2C" gate="J1" pin="2"/>
 </segment>
 <segment>
@@
 <wire x1="149.86" y1="96.52" x2="165.1" y2="96.52" width="0.1524" layer="91"/>
 <label x="152.4" y="96.52" size="1.778" layer="95"/>
-<pinref part="X4" gate="-4" pin="S"/>
-</segment>
-<segment>
+<pinref part="I2C" gate="J1" pin="1"/>
+</segment>
+<segment>

Commit message: I2c moved
So as not to interfere with other cables. other cables go up, i2c goes down to daughterboard
Parts:
- X3: value SCHLUESSELSPERRE -> SCHL-SPERRE
Changed lines of the file:
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@@
 <?xml version="1.0" encoding="utf-8"?>
 <!DOCTYPE eagle SYSTEM "eagle.dtd">
-<eagle version="7.7.0">
+<eagle version="7.6.0">
 <drawing>
 <settings>
@@
 <part name="X1" library="con-molex" deviceset="22-23-2041" device="" value="TASTENSPERRE1"/>
 <part name="X2" library="con-molex" deviceset="22-23-2041" device="" value="TASTENSPERRE2"/>
-<part name="X3" library="con-molex" deviceset="22-23-2021" device="" value="SCHLUESSELSPERRE"/>
+<part name="X3" library="con-molex" deviceset="22-23-2021" device="" value="SCHL-SPERRE"/>
 <part name="IC3" library="uln-udn" deviceset="ULN2803A" device="DIL18" value="ULN2803"/>
 <part name="GND13" library="supply1" deviceset="GND" device=""/>

Commit message: last update for mfg
Parts:
- added R1, R2: 4K7, resistor:R-EU_0207/7
Connections:
- net +5V: now also R1.2, R2.2
- net SCL: now also R1.1
- net SDA: now also R2.1
Changed lines of the file:
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@@
 <part name="GND16" library="supply1" deviceset="GND" device=""/>
 <part name="I2C" library="SparkFun-Connectors" deviceset="CONN_04" device="JST-PTH-VERT"/>
+<part name="R1" library="resistor" deviceset="R-EU_" device="0207/7" value="4K7"/>
+<part name="R2" library="resistor" deviceset="R-EU_" device="0207/7" value="4K7"/>
+<part name="P+1" library="supply1" deviceset="+5V" device=""/>
+<part name="P+6" library="supply1" deviceset="+5V" device=""/>
 </parts>
 <sheets>
@@
 <instance part="GND16" gate="1" x="-68.58" y="10.16"/>
 <instance part="I2C" gate="J1" x="170.18" y="99.06" rot="MR0"/>
+<instance part="R1" gate="G$1" x="147.32" y="111.76" rot="R90"/>
+<instance part="R2" gate="G$1" x="139.7" y="111.76" rot="R90"/>
+<instance part="P+1" gate="1" x="139.7" y="121.92"/>
+<instance part="P+6" gate="1" x="147.32" y="121.92"/>
 </instances>
 <busses>
@@
 <label x="152.4" y="88.9" size="1.778" layer="95"/>
 </segment>
+<segment>
+<pinref part="P+1" gate="1" pin="+5V"/>
+<pinref part="R2" gate="G$1" pin="2"/>
+<wire x1="139.7" y1="119.38" x2="139.7" y2="116.84" width="0.1524" layer="91"/>
+</segment>
+<segment>
+<pinref part="P+6" gate="1" pin="+5V"/>
+<pinref part="R1" gate="G$1" pin="2"/>
+<wire x1="147.32" y1="119.38" x2="147.32" y2="116.84" width="0.1524" layer="91"/>
+</segment>
 </net>
 <net name="LN_TX" class="0">
@@
 </segment>
 <segment>
-<wire x1="149.86" y1="99.06" x2="165.1" y2="99.06" width="0.1524" layer="91"/>
-<label x="152.4" y="99.06" size="1.778" layer="95"/>
+<wire x1="132.08" y1="99.06" x2="139.7" y2="99.06" width="0.1524" layer="91"/>
+<label x="132.08" y="99.06" size="1.778" layer="95"/>
 <pinref part="I2C" gate="J1" pin="2"/>
+<pinref part="R2" gate="G$1" pin="1"/>
+<wire x1="139.7" y1="99.06" x2="165.1" y2="99.06" width="0.1524" layer="91"/>
+<wire x1="139.7" y1="106.68" x2="139.7" y2="99.06" width="0.1524" layer="91"/>
+<junction x="139.7" y="99.06"/>
 </segment>
 <segment>
@@
 </segment>
 <segment>
-<wire x1="149.86" y1="96.52" x2="165.1" y2="96.52" width="0.1524" layer="91"/>
-<label x="152.4" y="96.52" size="1.778" layer="95"/>
+<wire x1="132.08" y1="96.52" x2="147.32" y2="96.52" width="0.1524" layer="91"/>
+<label x="132.08" y="96.52" size="1.778" layer="95"/>
 <pinref part="I2C" gate="J1" pin="1"/>
-</segment>
-<segment>
+<pinref part="R1" gate="G$1" pin="1"/>
+<wire x1="147.32" y1="96.52" x2="165.1" y2="96.52" width="0.1524" layer="91"/>
+<wire x1="147.32" y1="106.68" x2="147.32" y2="96.52" width="0.1524" layer="91"/>
+<junction x="147.32" y="96.52"/>
+</segment>
+<segment>
