File: hw/felderblock/Felderblock_Grundplatine.sch (EAGLE design)
At the start: 54 parts, among them IC2 LM2936, IC3 ULN2803, IC4 MCP2300X/P, J1 RJ11, J2 RJ11, M1 ARDUINO-NANO-3.0, T2 BC337, X1 TASTENSPERRE1, X2 TASTENSPERRE2, X3 SCHL-SPERRE, X5 ANSCHALTER

Commit message: LED 10mm updated
changes:
- footprint 10mm LED
- INT not connected to GND (=output)
Parts:
- LED1, LED2, LED3, LED4: device SparkFun-LED:LED10MM -> led:LED10MM
Connections:
- removed net N$19: IC3.I8
- removed net N$27: IC3.O8
- net GND: no longer IC4.INT
Changed lines of the file:
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@@
 <part name="GND9" library="supply1" deviceset="GND" device=""/>
 <part name="P+3" library="supply1" deviceset="+5V" device=""/>
-<part name="LED1" library="SparkFun-LED" deviceset="LED" device="10MM"/>
-<part name="LED2" library="SparkFun-LED" deviceset="LED" device="10MM"/>
-<part name="LED3" library="SparkFun-LED" deviceset="LED" device="10MM"/>
-<part name="LED4" library="SparkFun-LED" deviceset="LED" device="10MM"/>
+<part name="LED1" library="led" deviceset="LED" device="10MM"/>
+<part name="LED2" library="led" deviceset="LED" device="10MM"/>
+<part name="LED3" library="led" deviceset="LED" device="10MM"/>
+<part name="LED4" library="led" deviceset="LED" device="10MM"/>
 <part name="R11" library="resistor" deviceset="R-EU_" device="0207/7" value="1k"/>
 <part name="R12" library="resistor" deviceset="R-EU_" device="0207/7" value="1k"/>
@@
 <instance part="GND9" gate="1" x="25.4" y="124.46"/>
 <instance part="P+3" gate="1" x="33.02" y="200.66"/>
-<instance part="LED1" gate="D1" x="91.44" y="190.5" rot="R90"/>
-<instance part="LED2" gate="D1" x="91.44" y="175.26" rot="R90"/>
-<instance part="LED3" gate="D1" x="91.44" y="160.02" rot="R90"/>
-<instance part="LED4" gate="D1" x="91.44" y="144.78" rot="R90"/>
+<instance part="LED1" gate="G$1" x="91.44" y="190.5" rot="R90"/>
+<instance part="LED2" gate="G$1" x="91.44" y="175.26" rot="R90"/>
+<instance part="LED3" gate="G$1" x="91.44" y="160.02" rot="R90"/>
+<instance part="LED4" gate="G$1" x="91.44" y="144.78" rot="R90"/>
 <instance part="R11" gate="G$1" x="78.74" y="190.5"/>
 <instance part="R12" gate="G$1" x="78.74" y="175.26"/>
@@
 <pinref part="GND10" gate="1" pin="GND"/>
 <wire x1="101.6" y1="132.08" x2="101.6" y2="144.78" width="0.1524" layer="91"/>
-<pinref part="LED4" gate="D1" pin="C"/>
+<pinref part="LED4" gate="G$1" pin="C"/>
 <wire x1="101.6" y1="144.78" x2="96.52" y2="144.78" width="0.1524" layer="91"/>
-<pinref part="LED3" gate="D1" pin="C"/>
+<pinref part="LED3" gate="G$1" pin="C"/>
 <wire x1="96.52" y1="160.02" x2="101.6" y2="160.02" width="0.1524" layer="91"/>
 <wire x1="101.6" y1="160.02" x2="101.6" y2="144.78" width="0.1524" layer="91"/>
 <junction x="101.6" y="144.78"/>
-<pinref part="LED2" gate="D1" pin="C"/>
+<pinref part="LED2" gate="G$1" pin="C"/>
 <wire x1="96.52" y1="175.26" x2="101.6" y2="175.26" width="0.1524" layer="91"/>
 <wire x1="101.6" y1="175.26" x2="101.6" y2="160.02" width="0.1524" layer="91"/>
 <junction x="101.6" y="160.02"/>
-<pinref part="LED1" gate="D1" pin="C"/>
+<pinref part="LED1" gate="G$1" pin="C"/>
 <wire x1="96.52" y1="190.5" x2="101.6" y2="190.5" width="0.1524" layer="91"/>
 <wire x1="101.6" y1="190.5" x2="101.6" y2="175.26" width="0.1524" layer="91"/>
@@
 <pinref part="IC4" gate="G$1" pin="/RST"/>
 <wire x1="137.16" y1="76.2" x2="129.54" y2="76.2" width="0.1524" layer="91"/>
-<pinref part="IC4" gate="G$1" pin="INT"/>
-<wire x1="137.16" y1="71.12" x2="129.54" y2="71.12" width="0.1524" layer="91"/>
-<wire x1="129.54" y1="76.2" x2="129.54" y2="71.12" width="0.1524" layer="91"/>
 <junction x="129.54" y="76.2"/>
-<junction x="129.54" y="71.12"/>
-<wire x1="129.54" y1="71.12" x2="129.54" y2="55.88" width="0.1524" layer="91"/>
+<wire x1="129.54" y1="76.2" x2="129.54" y2="55.88" width="0.1524" layer="91"/>
 <pinref part="IC4" gate="G$1" pin="A2"/>
 <wire x1="137.16" y1="53.34" x2="129.54" y2="53.34" width="0.1524" layer="91"/>
@@
 <wire x1="-170.18" y1="27.94" x2="-149.86" y2="27.94" width="0.1524" layer="91"/>
 <pinref part="R16" gate="G$1" pin="1"/>
+<label x="-167.64" y="27.94" size="1.778" layer="95"/>
 </segment>
 </net>
@@
 <segment>
 <pinref part="R11" gate="G$1" pin="2"/>
-<pinref part="LED1" gate="D1" pin="A"/>
+<pinref part="LED1" gate="G$1" pin="A"/>
 <wire x1="83.82" y1="190.5" x2="88.9" y2="190.5" width="0.1524" layer="91"/>
 </segment>
@@
 <segment>
 <pinref part="R12" gate="G$1" pin="2"/>
-<pinref part="LED2" gate="D1" pin="A"/>
+<pinref part="LED2" gate="G$1" pin="A"/>
 <wire x1="83.82" y1="175.26" x2="88.9" y2="175.26" width="0.1524" layer="91"/>
 </segment>
@@
 <segment>
 <pinref part="R13" gate="G$1" pin="2"/>
-<pinref part="LED3" gate="D1" pin="A"/>
+<pinref part="LED3" gate="G$1" pin="A"/>
 <wire x1="83.82" y1="160.02" x2="88.9" y2="160.02" width="0.1524" layer="91"/>
 </segment>
@@
 <segment>
 <pinref part="R14" gate="G$1" pin="2"/>
-<pinref part="LED4" gate="D1" pin="A"/>
+<pinref part="LED4" gate="G$1" pin="A"/>
 <wire x1="83.82" y1="144.78" x2="88.9" y2="144.78" width="0.1524" layer="91"/>
 </segment>
@@
 </segment>
 </net>
-<net name="N$19" class="0">
-<segment>
-<pinref part="IC3" gate="G$1" pin="I8"/>
-<wire x1="27.94" y1="60.96" x2="43.18" y2="60.96" width="0.1524" layer="91"/>
-<label x="27.94" y="60.96" size="1.778" layer="95"/>
-</segment>
-</net>
-<net name="N$27" class="0">
-<segment>
-<pinref part="IC3" gate="G$1" pin="O8"/>
-<wire x1="83.82" y1="60.96" x2="68.58" y2="60.96" width="0.1524" layer="91"/>
-<label x="71.12" y="60.96" size="1.778" layer="95"/>
-</segment>
-</net>
 <net name="MI_FWD" class="0">
 <segment>
@@
 </sheet>
 </sheets>
+<errors>
+</errors>
 </schematic>
 </drawing>
