File: hw/felderblock/Felderblock_Hebelplatine.sch (EAGLE design)
At the start: 35 parts, among them IC3 MCP23017SP, X1 I2C-1, X4 I2C-2

Commit message: changed I2C connectors
Parts:
- removed X1: I2C-1, con-molex:22-23-2041
- removed X4: I2C-2, con-molex:22-23-2041
- added I2C-1, I2C-2: (no value), SparkFun-Connectors:CONN_04JST-PTH-VERT
Connections:
- net +5V: now also I2C-1.3, I2C-2.3; no longer X1-2.S, X4-2.S
- net GND: now also I2C-1.4, I2C-2.4; no longer X1-1.S, X4-1.S
- net SCL: now also I2C-1.1, I2C-2.1; no longer X1-4.S, X4-4.S
- net SDA: now also I2C-1.2, I2C-2.2; no longer X1-3.S, X4-3.S
Changed lines of the file:
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@@
 <?xml version="1.0" encoding="utf-8"?>
 <!DOCTYPE eagle SYSTEM "eagle.dtd">
-<eagle version="7.3.0">
+<eagle version="7.7.0">
 <drawing>
 <settings>
@@
 <part name="GND13" library="supply1" deviceset="GND" device=""/>
 <part name="P+5" library="supply1" deviceset="+5V" device=""/>
-<part name="X4" library="con-molex" deviceset="22-23-2041" device="" value="I2C-2"/>
 <part name="H1" library="holes" deviceset="MOUNT-HOLE" device="3.2"/>
 <part name="H2" library="holes" deviceset="MOUNT-HOLE" device="3.2"/>
 <part name="H3" library="holes" deviceset="MOUNT-HOLE" device="3.2"/>
 <part name="H4" library="holes" deviceset="MOUNT-HOLE" device="3.2"/>
-<part name="X1" library="con-molex" deviceset="22-23-2041" device="" value="I2C-1"/>
+<part name="I2C-1" library="SparkFun-Connectors" deviceset="CONN_04" device="JST-PTH-VERT"/>
+<part name="I2C-2" library="SparkFun-Connectors" deviceset="CONN_04" device="JST-PTH-VERT"/>
 </parts>
 <sheets>
@@
 <instance part="GND13" gate="1" x="25.4" y="27.94"/>
 <instance part="P+5" gate="1" x="25.4" y="88.9"/>
-<instance part="X4" gate="-1" x="60.96" y="109.22"/>
-<instance part="X4" gate="-2" x="60.96" y="106.68"/>
-<instance part="X4" gate="-3" x="60.96" y="104.14"/>
-<instance part="X4" gate="-4" x="60.96" y="101.6"/>
 <instance part="H1" gate="G$1" x="17.78" y="10.16"/>
 <instance part="H2" gate="G$1" x="17.78" y="2.54"/>
 <instance part="H3" gate="G$1" x="17.78" y="-5.08"/>
 <instance part="H4" gate="G$1" x="17.78" y="-12.7"/>
-<instance part="X1" gate="-1" x="58.42" y="127"/>
-<instance part="X1" gate="-2" x="58.42" y="124.46"/>
-<instance part="X1" gate="-3" x="58.42" y="121.92"/>
-<instance part="X1" gate="-4" x="58.42" y="119.38"/>
+<instance part="I2C-1" gate="J1" x="60.96" y="121.92" rot="MR0"/>
+<instance part="I2C-2" gate="J1" x="63.5" y="104.14" rot="MR0"/>
 </instances>
 <busses>
@@
 <wire x1="43.18" y1="109.22" x2="58.42" y2="109.22" width="0.1524" layer="91"/>
 <label x="45.72" y="109.22" size="1.778" layer="95"/>
-<pinref part="X4" gate="-1" pin="S"/>
+<pinref part="I2C-2" gate="J1" pin="4"/>
 </segment>
 <segment>
 <wire x1="40.64" y1="127" x2="55.88" y2="127" width="0.1524" layer="91"/>
 <label x="43.18" y="127" size="1.778" layer="95"/>
-<pinref part="X1" gate="-1" pin="S"/>
+<pinref part="I2C-1" gate="J1" pin="4"/>
 </segment>
 </net>
@@
 <wire x1="43.18" y1="106.68" x2="58.42" y2="106.68" width="0.1524" layer="91"/>
 <label x="45.72" y="106.68" size="1.778" layer="95"/>
-<pinref part="X4" gate="-2" pin="S"/>
+<pinref part="I2C-2" gate="J1" pin="3"/>
 </segment>
 <segment>
 <wire x1="40.64" y1="124.46" x2="55.88" y2="124.46" width="0.1524" layer="91"/>
 <label x="43.18" y="124.46" size="1.778" layer="95"/>
-<pinref part="X1" gate="-2" pin="S"/>
+<pinref part="I2C-1" gate="J1" pin="3"/>
 </segment>
 </net>
@@
 <wire x1="43.18" y1="104.14" x2="58.42" y2="104.14" width="0.1524" layer="91"/>
 <label x="45.72" y="104.14" size="1.778" layer="95"/>
-<pinref part="X4" gate="-3" pin="S"/>
+<pinref part="I2C-2" gate="J1" pin="2"/>
 </segment>
 <segment>
 <wire x1="40.64" y1="121.92" x2="55.88" y2="121.92" width="0.1524" layer="91"/>
 <label x="43.18" y="121.92" size="1.778" layer="95"/>
-<pinref part="X1" gate="-3" pin="S"/>
+<pinref part="I2C-1" gate="J1" pin="2"/>
 </segment>
 </net>
@@
 <wire x1="43.18" y1="101.6" x2="58.42" y2="101.6" width="0.1524" layer="91"/>
 <label x="45.72" y="101.6" size="1.778" layer="95"/>
-<pinref part="X4" gate="-4" pin="S"/>
+<pinref part="I2C-2" gate="J1" pin="1"/>
 </segment>
 <segment>
 <wire x1="40.64" y1="119.38" x2="55.88" y2="119.38" width="0.1524" layer="91"/>
 <label x="43.18" y="119.38" size="1.778" layer="95"/>
-<pinref part="X1" gate="-4" pin="S"/>
-</segment>
-</net>
+<pinref part="I2C-1" gate="J1" pin="1"/>
+</segment>
+</net>

Commit message: changed holes for switches to oval ones
Parts:
- FS1-5, FS2-6, FS3-7, FS4-8: device Jens:SW_2POL_ON-OFF-ONOVAL -> Jens:SW_2POL_ON-OFF-ONLANGLOCH
Changed lines of the file:
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@@
 <grid distance="0.1" unitdist="inch" unit="inch" style="lines" multiple="1" display="no" altdistance="0.01" altunitdist="inch" altunit="inch"/>
 <layers>
-<layer number="1" name="Top" color="4" fill="1" visible="no" active="no"/>
-<layer number="16" name="Bottom" color="1" fill="1" visible="no" active="no"/>
-<layer number="17" name="Pads" color="2" fill="1" visible="no" active="no"/>
-<layer number="18" name="Vias" color="2" fill="1" visible="no" active="no"/>
-<layer number="19" name="Unrouted" color="6" fill="1" visible="no" active="no"/>
-<layer number="20" name="Dimension" color="24" fill="1" visible="no" active="no"/>
-<layer number="21" name="tPlace" color="16" fill="1" visible="no" active="no"/>
-<layer number="22" name="bPlace" color="14" fill="1" visible="no" active="no"/>
-<layer number="23" name="tOrigins" color="15" fill="1" visible="no" active="no"/>
-<layer number="24" name="bOrigins" color="15" fill="1" visible="no" active="no"/>
-<layer number="25" name="tNames" color="7" fill="1" visible="no" active="no"/>
-<layer number="26" name="bNames" color="7" fill="1" visible="no" active="no"/>
-<layer number="27" name="tValues" color="7" fill="1" visible="no" active="no"/>
-<layer number="28" name="bValues" color="7" fill="1" visible="no" active="no"/>
+<layer number="1" name="Top" color="4" fill="1" visible="yes" active="no"/>
+<layer number="16" name="Bottom" color="1" fill="1" visible="yes" active="no"/>
+<layer number="17" name="Pads" color="2" fill="1" visible="yes" active="no"/>
+<layer number="18" name="Vias" color="2" fill="1" visible="yes" active="no"/>
+<layer number="19" name="Unrouted" color="6" fill="1" visible="yes" active="no"/>
+<layer number="20" name="Dimension" color="15" fill="1" visible="yes" active="no"/>
+<layer number="21" name="tPlace" color="7" fill="1" visible="yes" active="no"/>
+<layer number="22" name="bPlace" color="7" fill="1" visible="yes" active="no"/>
+<layer number="23" name="tOrigins" color="15" fill="1" visible="yes" active="no"/>
+<layer number="24" name="bOrigins" color="15" fill="1" visible="yes" active="no"/>
+<layer number="25" name="tNames" color="7" fill="1" visible="yes" active="no"/>
+<layer number="26" name="bNames" color="7" fill="1" visible="yes" active="no"/>
+<layer number="27" name="tValues" color="7" fill="1" visible="yes" active="no"/>
+<layer number="28" name="bValues" color="7" fill="1" visible="yes" active="no"/>
 <layer number="29" name="tStop" color="7" fill="3" visible="no" active="no"/>
 <layer number="30" name="bStop" color="7" fill="6" visible="no" active="no"/>
@@
 <layer number="35" name="tGlue" color="7" fill="4" visible="no" active="no"/>
 <layer number="36" name="bGlue" color="7" fill="5" visible="no" active="no"/>
-<layer number="37" name="tTest" color="7" fill="1" visible="no" active="no"/>
-<layer number="38" name="bTest" color="7" fill="1" visible="no" active="no"/>
+<layer number="37" name="tTest" color="7" fill="1" visible="yes" active="no"/>
+<layer number="38" name="bTest" color="7" fill="1" visible="yes" active="no"/>
 <layer number="39" name="tKeepout" color="4" fill="11" visible="no" active="no"/>
 <layer number="40" name="bKeepout" color="1" fill="11" visible="no" active="no"/>
@@
 <layer number="44" name="Drills" color="7" fill="1" visible="no" active="no"/>
 <layer number="45" name="Holes" color="7" fill="1" visible="no" active="no"/>
-<layer number="46" name="Milling" color="3" fill="1" visible="no" active="no"/>
-<layer number="47" name="Measures" color="7" fill="1" visible="no" active="no"/>
-<layer number="48" name="Document" color="7" fill="1" visible="no" active="no"/>
-<layer number="49" name="Reference" color="13" fill="1" visible="no" active="no"/>
-<layer number="50" name="dxf" color="7" fill="1" visible="no" active="no"/>
-<layer number="51" name="tDocu" color="6" fill="1" visible="no" active="no"/>
-<layer number="52" name="bDocu" color="7" fill="1" visible="no" active="no"/>
-<layer number="53" name="tGND_GNDA" color="7" fill="9" visible="no" active="no"/>
-<layer number="54" name="bGND_GNDA" color="1" fill="9" visible="no" active="no"/>
-<layer number="56" name="wert" color="7" fill="1" visible="no" active="no"/>
-<layer number="57" name="tCAD" color="7" fill="1" visible="no" active="no"/>
-<layer number="58" name="bCAD" color="7" fill="1" visible="no" active="no"/>
-<layer number="59" name="tCarbon" color="7" fill="1" visible="no" active="no"/>
-<layer number="60" name="bCarbon" color="7" fill="1" visible="no" active="no"/>
+<layer number="46" name="Milling" color="3" fill="1" visible="yes" active="no"/>
+<layer number="47" name="Measures" color="7" fill="1" visible="yes" active="no"/>
+<layer number="48" name="Document" color="7" fill="1" visible="yes" active="no"/>
+<layer number="49" name="Reference" color="7" fill="1" visible="yes" active="no"/>
+<layer number="50" name="dxf" color="7" fill="1" visible="yes" active="no"/>
+<layer number="51" name="tDocu" color="7" fill="1" visible="yes" active="no"/>
+<layer number="52" name="bDocu" color="7" fill="1" visible="yes" active="no"/>
+<layer number="53" name="tGND_GNDA" color="7" fill="9" visible="yes" active="no"/>
+<layer number="54" name="bGND_GNDA" color="1" fill="9" visible="yes" active="no"/>
+<layer number="56" name="wert" color="7" fill="1" visible="yes" active="no"/>
+<layer number="57" name="tCAD" color="7" fill="1" visible="yes" active="no"/>
+<layer number="58" name="bCAD" color="7" fill="1" visible="yes" active="no"/>
+<layer number="59" name="tCarbon" color="7" fill="1" visible="yes" active="no"/>
+<layer number="60" name="bCarbon" color="7" fill="1" visible="yes" active="no"/>
 <layer number="88" name="SimResults" color="9" fill="1" visible="no" active="yes"/>
 <layer number="89" name="SimProbes" color="9" fill="1" visible="no" active="yes"/>
@@
 </classes>
 <parts>
-<part name="FS1-5" library="Jens" deviceset="SW_2POL_ON-OFF-ON" device="OVAL"/>
-<part name="FS2-6" library="Jens" deviceset="SW_2POL_ON-OFF-ON" device="OVAL"/>
-<part name="FS3-7" library="Jens" deviceset="SW_2POL_ON-OFF-ON" device="OVAL"/>
-<part name="FS4-8" library="Jens" deviceset="SW_2POL_ON-OFF-ON" device="OVAL"/>
+<part name="FS1-5" library="Jens" deviceset="SW_2POL_ON-OFF-ON" device="LANGLOCH"/>
+<part name="FS2-6" library="Jens" deviceset="SW_2POL_ON-OFF-ON" device="LANGLOCH"/>
+<part name="FS3-7" library="Jens" deviceset="SW_2POL_ON-OFF-ON" device="LANGLOCH"/>
+<part name="FS4-8" library="Jens" deviceset="SW_2POL_ON-OFF-ON" device="LANGLOCH"/>
 <part name="R15" library="resistor" deviceset="R-EU_" device="0207/7" value="10k"/>
 <part name="R16" library="resistor" deviceset="R-EU_" device="0207/7" value="10k"/>

Commit message: some tuning
Parts:
- FS1-5, FS2-6, FS3-7, FS4-8: device Jens:SW_2POL_ON-OFF-ONLANGLOCH -> Jens:SW_2POL_ON-OFF-ONSOLDERPAD
Changed lines of the file:
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@@
 <?xml version="1.0" encoding="utf-8"?>
 <!DOCTYPE eagle SYSTEM "eagle.dtd">
-<eagle version="7.7.0">
+<eagle version="7.6.0">
 <drawing>
 <settings>
@@
 <grid distance="0.1" unitdist="inch" unit="inch" style="lines" multiple="1" display="no" altdistance="0.01" altunitdist="inch" altunit="inch"/>
 <layers>
-<layer number="1" name="Top" color="4" fill="1" visible="yes" active="no"/>
-<layer number="16" name="Bottom" color="1" fill="1" visible="yes" active="no"/>
-<layer number="17" name="Pads" color="2" fill="1" visible="yes" active="no"/>
-<layer number="18" name="Vias" color="2" fill="1" visible="yes" active="no"/>
-<layer number="19" name="Unrouted" color="6" fill="1" visible="yes" active="no"/>
-<layer number="20" name="Dimension" color="15" fill="1" visible="yes" active="no"/>
-<layer number="21" name="tPlace" color="7" fill="1" visible="yes" active="no"/>
-<layer number="22" name="bPlace" color="7" fill="1" visible="yes" active="no"/>
-<layer number="23" name="tOrigins" color="15" fill="1" visible="yes" active="no"/>
-<layer number="24" name="bOrigins" color="15" fill="1" visible="yes" active="no"/>
-<layer number="25" name="tNames" color="7" fill="1" visible="yes" active="no"/>
-<layer number="26" name="bNames" color="7" fill="1" visible="yes" active="no"/>
-<layer number="27" name="tValues" color="7" fill="1" visible="yes" active="no"/>
-<layer number="28" name="bValues" color="7" fill="1" visible="yes" active="no"/>
+<layer number="1" name="Top" color="4" fill="1" visible="no" active="no"/>
+<layer number="16" name="Bottom" color="1" fill="1" visible="no" active="no"/>
+<layer number="17" name="Pads" color="2" fill="1" visible="no" active="no"/>
+<layer number="18" name="Vias" color="2" fill="1" visible="no" active="no"/>
+<layer number="19" name="Unrouted" color="6" fill="1" visible="no" active="no"/>
+<layer number="20" name="Dimension" color="15" fill="1" visible="no" active="no"/>
+<layer number="21" name="tPlace" color="7" fill="1" visible="no" active="no"/>
+<layer number="22" name="bPlace" color="7" fill="1" visible="no" active="no"/>
+<layer number="23" name="tOrigins" color="15" fill="1" visible="no" active="no"/>
+<layer number="24" name="bOrigins" color="15" fill="1" visible="no" active="no"/>
+<layer number="25" name="tNames" color="7" fill="1" visible="no" active="no"/>
+<layer number="26" name="bNames" color="7" fill="1" visible="no" active="no"/>
+<layer number="27" name="tValues" color="7" fill="1" visible="no" active="no"/>
+<layer number="28" name="bValues" color="7" fill="1" visible="no" active="no"/>
 <layer number="29" name="tStop" color="7" fill="3" visible="no" active="no"/>
 <layer number="30" name="bStop" color="7" fill="6" visible="no" active="no"/>
@@
 <layer number="35" name="tGlue" color="7" fill="4" visible="no" active="no"/>
 <layer number="36" name="bGlue" color="7" fill="5" visible="no" active="no"/>
-<layer number="37" name="tTest" color="7" fill="1" visible="yes" active="no"/>
-<layer number="38" name="bTest" color="7" fill="1" visible="yes" active="no"/>
+<layer number="37" name="tTest" color="7" fill="1" visible="no" active="no"/>
+<layer number="38" name="bTest" color="7" fill="1" visible="no" active="no"/>
 <layer number="39" name="tKeepout" color="4" fill="11" visible="no" active="no"/>
 <layer number="40" name="bKeepout" color="1" fill="11" visible="no" active="no"/>
@@
 <layer number="44" name="Drills" color="7" fill="1" visible="no" active="no"/>
 <layer number="45" name="Holes" color="7" fill="1" visible="no" active="no"/>
-<layer number="46" name="Milling" color="3" fill="1" visible="yes" active="no"/>
-<layer number="47" name="Measures" color="7" fill="1" visible="yes" active="no"/>
-<layer number="48" name="Document" color="7" fill="1" visible="yes" active="no"/>
-<layer number="49" name="Reference" color="7" fill="1" visible="yes" active="no"/>
-<layer number="50" name="dxf" color="7" fill="1" visible="yes" active="no"/>
-<layer number="51" name="tDocu" color="7" fill="1" visible="yes" active="no"/>
-<layer number="52" name="bDocu" color="7" fill="1" visible="yes" active="no"/>
-<layer number="53" name="tGND_GNDA" color="7" fill="9" visible="yes" active="no"/>
-<layer number="54" name="bGND_GNDA" color="1" fill="9" visible="yes" active="no"/>
-<layer number="56" name="wert" color="7" fill="1" visible="yes" active="no"/>
-<layer number="57" name="tCAD" color="7" fill="1" visible="yes" active="no"/>
-<layer number="58" name="bCAD" color="7" fill="1" visible="yes" active="no"/>
-<layer number="59" name="tCarbon" color="7" fill="1" visible="yes" active="no"/>
-<layer number="60" name="bCarbon" color="7" fill="1" visible="yes" active="no"/>
+<layer number="46" name="Milling" color="3" fill="1" visible="no" active="no"/>
+<layer number="47" name="Measures" color="7" fill="1" visible="no" active="no"/>
+<layer number="48" name="Document" color="7" fill="1" visible="no" active="no"/>
+<layer number="49" name="Reference" color="7" fill="1" visible="no" active="no"/>
+<layer number="50" name="dxf" color="7" fill="1" visible="no" active="no"/>
+<layer number="51" name="tDocu" color="7" fill="1" visible="no" active="no"/>
+<layer number="52" name="bDocu" color="7" fill="1" visible="no" active="no"/>
+<layer number="53" name="tGND_GNDA" color="7" fill="9" visible="no" active="no"/>
+<layer number="54" name="bGND_GNDA" color="1" fill="9" visible="no" active="no"/>
+<layer number="56" name="wert" color="7" fill="1" visible="no" active="no"/>
+<layer number="57" name="tCAD" color="7" fill="1" visible="no" active="no"/>
+<layer number="58" name="bCAD" color="7" fill="1" visible="no" active="no"/>
+<layer number="59" name="tCarbon" color="7" fill="1" visible="no" active="no"/>
+<layer number="60" name="bCarbon" color="7" fill="1" visible="no" active="no"/>
 <layer number="88" name="SimResults" color="9" fill="1" visible="no" active="yes"/>
 <layer number="89" name="SimProbes" color="9" fill="1" visible="no" active="yes"/>
@@
 </classes>
 <parts>
-<part name="FS1-5" library="Jens" deviceset="SW_2POL_ON-OFF-ON" device="LANGLOCH"/>
-<part name="FS2-6" library="Jens" deviceset="SW_2POL_ON-OFF-ON" device="LANGLOCH"/>
-<part name="FS3-7" library="Jens" deviceset="SW_2POL_ON-OFF-ON" device="LANGLOCH"/>
-<part name="FS4-8" library="Jens" deviceset="SW_2POL_ON-OFF-ON" device="LANGLOCH"/>
+<part name="FS1-5" library="Jens" deviceset="SW_2POL_ON-OFF-ON" device="SOLDERPAD"/>
+<part name="FS2-6" library="Jens" deviceset="SW_2POL_ON-OFF-ON" device="SOLDERPAD"/>
+<part name="FS3-7" library="Jens" deviceset="SW_2POL_ON-OFF-ON" device="SOLDERPAD"/>
+<part name="FS4-8" library="Jens" deviceset="SW_2POL_ON-OFF-ON" device="SOLDERPAD"/>
 <part name="R15" library="resistor" deviceset="R-EU_" device="0207/7" value="10k"/>
 <part name="R16" library="resistor" deviceset="R-EU_" device="0207/7" value="10k"/>

Commit message: last check
Parts:
- FS1-5, FS2-6, FS3-7, FS4-8: device Jens:SW_2POL_ON-OFF-ONSOLDERPAD -> Jens:SW_2POL_ON-OFF-ONLANGLOCH
Changed lines of the file:
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@@
 </classes>
 <parts>
-<part name="FS1-5" library="Jens" deviceset="SW_2POL_ON-OFF-ON" device="SOLDERPAD"/>
-<part name="FS2-6" library="Jens" deviceset="SW_2POL_ON-OFF-ON" device="SOLDERPAD"/>
-<part name="FS3-7" library="Jens" deviceset="SW_2POL_ON-OFF-ON" device="SOLDERPAD"/>
-<part name="FS4-8" library="Jens" deviceset="SW_2POL_ON-OFF-ON" device="SOLDERPAD"/>
+<part name="FS1-5" library="Jens" deviceset="SW_2POL_ON-OFF-ON" device="LANGLOCH"/>
+<part name="FS2-6" library="Jens" deviceset="SW_2POL_ON-OFF-ON" device="LANGLOCH"/>
+<part name="FS3-7" library="Jens" deviceset="SW_2POL_ON-OFF-ON" device="LANGLOCH"/>
+<part name="FS4-8" library="Jens" deviceset="SW_2POL_ON-OFF-ON" device="LANGLOCH"/>
 <part name="R15" library="resistor" deviceset="R-EU_" device="0207/7" value="10k"/>
 <part name="R16" library="resistor" deviceset="R-EU_" device="0207/7" value="10k"/>
